File: Uroflow_PCB/Uroflow_PCB.sch (KiCad schematic (older format))
At the start: 21 parts, among them P1 USB_OTG, U1 ATmega32U4-AU, U2 MPX5010DP, U3 TPS55330, U4 MotorValve, Y1 Crystal

Commit message: Incremental
Parts:
- added D2, D3: D, Diodes_SMD:D_0603, symbol D
- added Q1, Q3: Q_NPN_BCE, TO_SOT_Packages_SMD:SOT-23, symbol Q_NPN_BCE
- added Q2, Q4: Q_PMOS_DGS, TO_SOT_Packages_SMD:SOT-23, symbol Q_PMOS_DGS
- added R10, R11, R7, R8, R9: 1k, Resistors_SMD:R_0603, symbol R
- added U5: HC-05, Pin_Headers:Pin_Header_Straight_1x06, symbol HC-05
- added U6: PUSH_BUTTON, Buttons_Switches_THT:PUSH_BUTTON_large, symbol PUSH_BUTTON
- C1, C2: value C_Small -> 10p; footprint (none) -> Capacitors_SMD:C_0603
- C3, C4, C5, C6, C7: footprint (none) -> Capacitors_SMD:C_0603
- D1: footprint (none) -> Diodes_SMD:D_0603
- L1: footprint (none) -> Inductors:Inductor_Taiyo-Yuden_MD-3030
- P1: footprint (none) -> Connectors:USB_Micro-B
- R1, R2: value R -> 22; footprint (none) -> Resistors_SMD:R_0603
- R3, R4, R5, R6: footprint (none) -> Resistors_SMD:R_0603
- U1: footprint (none) -> Housings_QFP:TQFP-44_10x10mm_Pitch0.8mm
- U2: footprint (none) -> Pin_Headers:Pin_Header_Straight_1x06
- U3: footprint (none) -> Housings_DFN_QFN:QFN-16-1EP_3x3mm_Pitch0.5mm
- U4: footprint (none) -> Pin_Headers:Pin_Header_Straight_1x03
- Y1: footprint (none) -> Crystals:ABM3
Connections:
- net 12V: now also Q2.1 (D), Q4.1 (D), R10.2, R8.2
- net GND: now also U4.1 (GND), D2.2 (A), D3.2 (A), Q1.3 (E), Q3.3 (E), R11.2, U5.4 (GND)
- net VCC: now also U5.5 (VCC), U6.1 (+)
- net CLOSE_PIN: now reaches U1.10 ((PDI/MOSI/PCINT2)PB2)
- net CLOSE_PIN: now also R9.2
- net RX: now reaches U1.20 ((RXD/INT2)PD2)
- net RX: now also U5.2 (RX)
- net TX: now reaches U1.21 ((TXD/INT3)PD3)
- net TX: now also U5.3 (TX)
- net BUTTON: now reaches U1.32 ((ICP3/CLK0/OC4A)PC7)
- net BUTTON: now also R11.1, U6.2 (-)
- net OPEN_PIN: now reaches U1.9 ((SCLK/PCINT1)PB1)
- net OPEN_PIN: now also R7.2
- net CLOSE: now reaches U4.2 (Close)
- net CLOSE: now also D3.1 (K), Q4.3 (S)
- net OPEN: now reaches U4.3 (Open)
- net OPEN: now also D2.1 (K), Q2.3 (S)
- new net: Q1.1 (B), R7.1
- new net: Q1.2 (C), Q2.2 (G), R8.1
- new net: Q3.1 (B), R9.1
- new net: Q3.2 (C), Q4.2 (G), R10.1
- no-connect marks 4 -> 8
Other:
- note added: "Bluetooth"
- note added: "Microcontroller"
- note added: "Power"
- note added: "Sensor"
- note added: "Valve"
- moved on the sheet: C1, C2, P1, R1, R2, U1, U2, U4, Y1
